File: StepUp.brd (EAGLE design)
At the start: 100 x 80 mm, 42 parts, among them IC1 TL494CN, Q1 IRFZ48Z, Q10 A733, Q2 IRFZ48Z, Q3 IRFZ48Z, Q4 IRFZ48Z, Q5 IRFZ48Z, Q6 IRFZ48Z, Q7 IRFZ48Z, Q8 IRFZ48Z, Q9 A733

Commit message: Use class C bridge as MOSFET driver
Parts:
- removed D3, D8: (no value), diode:D-2.5
- removed L1: 10µ, rcl:6000-XXXX-RC
- removed R13, R14: 150, rcl:0204V
- removed R15, R16: 1k, rcl:0207/10
- removed SV1: (no value), con-lstb:MA03-1
- removed SV4: (no value), con-lstb:MA04-1
- removed TR1: (no value), trafo:FL02-08
- added L2: 10µ, rcl:6000-XXXX-RC
- added Q11: BD139, transistor-power:TO126AV
- added Q12, Q14: IRFZ48Z, transistor-power:TO220BH
- added Q13: BD140, transistor-power:TO126AV
- added R5, R7: 470, rcl:0204V
- added R8: 27k, rcl:0204/7
- added R9: 1M6, rcl:0207/15
- added TR2: (no value), trafo:FL02-08
- C1: device rcl:E2,5-7 -> rcl:E2,5-5
- C2: value 100µ -> 1000µ
- C4, C7, C8: value (none) -> 3300µ; device rcl:E3,5-8 -> rcl:E5-8,5
- C5: device rcl:C025-040X050 -> rcl:C025-024X044
- Q10: value A733 -> BD140; device transistor-pnp:TO92 -> transistor-power:TO126AV
- Q9: value A733 -> BD139; device transistor-pnp:TO92 -> transistor-power:TO126AV
- R17, R6: value 18 -> 1
- SV3: device con-lstb:MA04-1 -> con-lstb:MA03-1
- moved C8 181.5 mm to (99.1, 43.2), turned to 180 degrees
- moved C7 166.0 mm to (99.1, 63.5), turned to 180 degrees
- moved SV3 155.2 mm to (-95.8, -65.5), turned to 0 degrees
- moved C4 145.7 mm to (99.1, 53.3), turned to 180 degrees
- moved R17 142.6 mm to (26.7, 66.0), turned to 180 degrees
- moved R6 131.4 mm to (26.7, 50.8), turned to 180 degrees
- moved Q5 33.1 mm to (38.1, 36.8)
- moved Q6 33.1 mm to (50.8, 36.8)
- moved Q7 33.1 mm to (63.5, 36.8)
- moved Q8 33.1 mm to (76.2, 36.8)
- moved Q9 24.7 mm to (22.9, 54.6)
- moved Q4 23.3 mm to (76.2, 52.1), turned to 180 degrees
- moved Q3 22.8 mm to (63.5, 52.1), turned to 180 degrees
- moved Q2 22.3 mm to (50.8, 52.1), turned to 180 degrees
- moved R4 21.9 mm to (14.0, 45.7), turned to 180 degrees
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Connections:
- removed net N$19: C3.-, C4.+, C6.-, C7.+, C8.+, C9.-, SV2.2, TR1.6, TR1.7
- removed net N$22: C4.-, C7.-, C8.-, D6.A, D7.A, SV2.3
- removed net N$23: D3.A, IC1.9, Q9.2, R15.2
- removed net N$24: D8.A, IC1.10, Q10.2, R16.1
- removed net N$25: C3.+, C6.+, C9.+, D4.C, D5.C, SV2.1
- removed net N$26: D3.C, Q9.1, R13.2, R17.2
- removed net N$29: R17.1, SV3.2
- removed net N$30: D8.C, Q10.1, R14.1, R6.1
- removed net N$31: R6.2, SV3.3
- removed net N$32: C2.-, Q1.S, Q2.S, Q3.S, Q4.S, Q5.S, Q6.S, Q7.S, Q8.S, SV1.1, SV1.2, SV4.1
- new net +12V: C2.+, IC1.12, Q11.C, Q9.C, R4.2, SV3.2
- new net GND: C2.-, C3.-, C4.-, C5.2, C6.-, C7.-, C8.-, C9.-, D6.A, D7.A, IC1.1, IC1.7, Q1.S, Q10.C, Q12.S, Q13.C, Q14.S, Q2.S, Q3.S, Q4.S, Q5.S, Q6.S, Q7.S, Q8.S, R2.1, R3.2, R5.1, R7.1, R8.1, SV2.2, SV2.3, SV3.1
- new net N$12: IC1.10, Q11.B, Q13.B, R5.2
- new net N$16: Q10.E, Q9.E, R6.2
- new net N$17: IC1.9, Q10.B, Q9.B, R7.2
- new net N$8: Q11.E, Q13.E, R17.2
- new net V+: C3.+, C6.+, C9.+, D4.C, D5.C, R9.2, SV2.1
- net N$1: now also L2.1, SV3.3; no longer C2.+, L1.1, SV1.3
- net N$13: now also Q14.G, R6.1; no longer SV4.3
- net N$20: now also TR2.8; no longer TR1.8
- net N$21: now also TR2.5; no longer TR1.5
- net N$27: now also Q14.D, TR2.4; no longer TR1.4
- net N$28: now also Q12.D, TR2.1; no longer TR1.1
- net N$33: now also C4.+, C7.+, C8.+, L2.2, TR2.2, TR2.3; no longer L1.2, SV4.4, TR1.2, TR1.3
- net N$4: now also R8.2, R9.1; no longer C5.2, IC1.1, IC1.7, Q10.3, Q9.3, R13.1, R14.2, R15.1, R16.2, R2.1, R3.2, SV3.1
- net N$7: now also TR2.6, TR2.7; no longer IC1.12, R4.2, SV3.4
- net N$9: now also Q12.G, R17.1; no longer SV4.2
Routing:
- net GND: track 0.00 -> 264.2 mm, vias 0 -> 2
- net N$28: track 0.00 -> 185.4 mm, vias 0 -> 2
- net N$9: track 0.00 -> 165.1 mm, vias 0 -> 12
- net N$27: track 6.60 -> 167.6 mm
- net N$13: track 48.3 -> 188.0 mm, vias 6 -> 12
- net N$32: track 66.0 -> 0.00 mm
- net +12V: track 0.00 -> 66.0 mm, vias 0 -> 2
- net N$33: track 0.00 -> 35.6 mm
- net N$12: track 0.00 -> 31.0 mm
- net N$4: track 94.0 -> 121.9 mm, vias 4 -> 0
- net N$23: track 23.5 -> 0.00 mm
- net N$24: track 19.7 -> 0.00 mm
- net N$17: track 0.00 -> 13.2 mm
- net N$1: track 12.7 -> 0.00 mm
- net N$7: track 12.7 -> 0.00 mm
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Other:
- board size 100 x 80 mm -> 162.5 x 83.8 mm
