File: StepUp.sch (EAGLE design)
At the start: 42 parts, among them IC1 TL494CN, Q1 IRFZ48Z, Q10 A733, Q2 IRFZ48Z, Q3 IRFZ48Z, Q4 IRFZ48Z, Q5 IRFZ48Z, Q6 IRFZ48Z, Q7 IRFZ48Z, Q8 IRFZ48Z, Q9 A733

Commit message: Use class C bridge as MOSFET driver
Parts:
- removed D3, D8: (no value), diode:DIODE-D-2.5
- removed L1: 10µ, rcl:L-US6000-XXX-RC
- removed R13, R14: 150, rcl:R-EU_0204/2V
- removed R15, R16: 1k, rcl:R-EU_0207/10
- removed SV1: (no value), con-lstb:MA03-1
- removed SV4: (no value), con-lstb:MA04-1
- removed TR1: (no value), trafo:FL02
- added L2: 10µ, rcl:L-US6000-XXX-RC
- added Q11: BD139, transistor-power:BD139
- added Q12, Q14: IRFZ48Z, transistor-power:IRFZ48Z
- added Q13: BD140, transistor-power:BD140
- added R5, R7: 470, rcl:R-EU_0204/2V
- added R8: 27k, rcl:R-EU_0204/7
- added R9: 1M6, rcl:R-EU_0207/15
- added TR2: (no value), trafo:FL02
- C1: device rcl:CPOL-EUE2.5-7 -> rcl:CPOL-EUE2.5-5
- C2: value 100µ -> 1000µ
- C4, C7, C8: value (none) -> 3300µ; device rcl:CPOL-EUE3.5-8 -> rcl:CPOL-EUE5-8.5
- C5: device rcl:C-EU025-040X050 -> rcl:C-EU025-024X044
- Q10: value A733 -> BD140; device transistor-pnp:BC214 -> transistor-power:BD140
- Q9: value A733 -> BD139; device transistor-pnp:BC214 -> transistor-power:BD139
- R17, R6: value 18 -> 1
- SV3: device con-lstb:MA04-1 -> con-lstb:MA03-1
Connections:
- removed net N$19: C3.-, C4.+, C6.-, C7.+, C8.+, C9.-, SV2.2, TR1.6, TR1.7
- removed net N$22: C4.-, C7.-, C8.-, D6.A, D7.A, SV2.3
- removed net N$23: D3.A, IC1.E1, Q9.B, R15.2
- removed net N$24: D8.A, IC1.E2, Q10.B, R16.1
- removed net N$25: C3.+, C6.+, C9.+, D4.C, D5.C, SV2.1
- removed net N$26: D3.C, Q9.E, R13.2, R17.2
- removed net N$29: R17.1, SV3.2
- removed net N$30: D8.C, Q10.E, R14.1, R6.1
- removed net N$31: R6.2, SV3.3
- removed net N$32: C2.-, Q1.S, Q2.S, Q3.S, Q4.S, Q5.S, Q6.S, Q7.S, Q8.S, SV1.1, SV1.2, SV4.1
- new net +12V: C2.+, IC1.VCC, Q11.C, Q9.C, R4.2, SV3.2
- new net GND: C2.-, C3.-, C4.-, C5.2, C6.-, C7.-, C8.-, C9.-, D6.A, D7.A, IC1.+I1, IC1.GND, Q1.S, Q10.C, Q12.S, Q13.C, Q14.S, Q2.S, Q3.S, Q4.S, Q5.S, Q6.S, Q7.S, Q8.S, R2.1, R3.2, R5.1, R7.1, R8.1, SV2.2, SV2.3, SV3.1
- new net N$12: IC1.E2, Q11.B, Q13.B, R5.2
- new net N$16: Q10.E, Q9.E, R6.2
- new net N$17: IC1.E1, Q10.B, Q9.B, R7.2
- new net N$8: Q11.E, Q13.E, R17.2
- new net V+: C3.+, C6.+, C9.+, D4.C, D5.C, R9.2, SV2.1
- net N$1: now also L2.1, SV3.3; no longer C2.+, L1.1, SV1.3
- net N$13: now also Q14.G, R6.1; no longer SV4.3
- net N$20: now also TR2.8; no longer TR1.8
- net N$21: now also TR2.5; no longer TR1.5
- net N$27: now also Q14.D, TR2.4; no longer TR1.4
- net N$28: now also Q12.D, TR2.1; no longer TR1.1
- net N$33: now also C4.+, C7.+, C8.+, L2.2, TR2.2, TR2.3; no longer L1.2, SV4.4, TR1.2, TR1.3
- net N$4: now also R8.2, R9.1; no longer C5.2, IC1.+I1, IC1.GND, Q10.C, Q9.C, R13.1, R14.2, R15.1, R16.2, R2.1, R3.2, SV3.1
- net N$7: now also TR2.6, TR2.7; no longer IC1.VCC, R4.2, SV3.4
- net N$9: now also Q12.G, R17.1; no longer SV4.2
Other:
- moved on the sheet: C2, C3, C4, C6, C7, C8, C9, D4, D5, D6, D7, Q1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
